File: TEJ4M-Unit-4-08/TEJ4M-Unit-4-08.kicad_sch (KiCad schematic)
At the start: 13 parts, among them U1 ADG417BN, U2 ADG417BN, U3 4001, U4 74LS08, U5 74AHC04, U6 74LS08, U7 4001

Commit message: Add files via upload
Parts:
- added H1, H2, H3, H4: MountingHole, MountingHole:MountingHole_2.5mm, symbol Mechanical:MountingHole
- added J1, J2, J3, J4: Conn_01x03_Socket, Connector_PinSocket_1.27mm:PinSocket_1x03_P1.27mm_Vertical, symbol Connector:Conn_01x03_Socket
- D3: renamed from D1; footprint (none) -> LED_THT:LED_D3.0mm_Horizontal_O1.27mm_Z2.0mm
- D4: renamed from D2; footprint (none) -> LED_THT:LED_D3.0mm_Horizontal_O1.27mm_Z2.0mm
- R1: renamed from R3; footprint (none) -> Resistor_THT:R_Axial_DIN0207_L6.3mm_D2.5mm_P7.62mm_Horizontal
- R2: renamed from R1; footprint (none) -> Resistor_THT:R_Axial_DIN0207_L6.3mm_D2.5mm_P7.62mm_Horizontal
- R3: renamed from R2; footprint (none) -> Resistor_THT:R_Axial_DIN0207_L6.3mm_D2.5mm_P7.62mm_Horizontal
- R4: footprint (none) -> Resistor_THT:R_Axial_DIN0207_L6.3mm_D2.5mm_P7.62mm_Horizontal
- U1: renamed from U2; footprint Package_DIP:DIP-8_W7.62mm -> Button_Switch_THT:SW_PUSH_6mm
- U2: renamed from U1; footprint Package_DIP:DIP-8_W7.62mm -> Button_Switch_THT:SW_PUSH_6mm
- U3: renamed from U5; footprint (none) -> Package_DIP:DIP-8_W7.62mm
- U4: renamed from U6; footprint (none) -> Package_DIP:DIP-8_W7.62mm
- U5: renamed from U4; footprint (none) -> Package_DIP:DIP-8_W7.62mm
- U6: renamed from U7; footprint (none) -> Package_DIP:DIP-8_W7.62mm
- U7: renamed from U3; footprint (none) -> Package_DIP:DIP-8_W7.62mm
Connections:
- net at R2.1, U4.1, U5.2: now also U2.2; no longer U2.8
- net at R1.1, U3.1, U4.2: now also U1.2; no longer U1.8
- net +5V: no longer names the net of U2.1
- net +5V: now also J1.2 (Pin_2); no longer U1.1
- removed net GND: R1.2, R2.2, R3.2, R4.2
- new net: J1.1 (Pin_1), U1.1
- new net: J2.2 (Pin_2), R2.2
- new net: J2.1 (Pin_1), R1.2
- new net: J4.1 (Pin_1), R3.2
- new net: J4.2 (Pin_2), R4.2
Other:
- note added: "Curtis Edwards TEJ4M Unit-4-08"
- note removed: "Curtis Edwards TEJ4M Unit-2-08"
